File: pcb/serialsentinel.kicad_pcb (KiCad board)
At the start: 4 copper layers, 73.2 x 64.4 mm, 39 parts, among them J2 Bus_PCI_Express_x1, J3 REL1, J4 REL1, J5 REL2, J6 REL2, K2 G6K-2F-Y DC3, K3 G6K-2F-Y DC3, Q2 MMBT3904, Q3 MMBT3904, Q4 MMBT3904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

Commit message: tweak
Routing:
- net Net-(Q2-B): track 13.1 -> 13.9 mm
Other:
- board text added: "<<hash>>"
- board text added: "JLCJLCJLCJLC"
- board text added: "github.com/gcormier/serialsentinel v1"
- board text removed: "github.com/gcormier/serialsentinel"
Changed lines of the file:
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@@
 		(layer "F.Fab")
 	)
-	(gr_text "github.com/gcormier/serialsentinel"
+	(gr_text "<<hash>>"
+		(at 25.829563 89.575461 90)
+		(layer "F.SilkS")
+		(effects
+			(font
+				(size 1 1)
+				(thickness 0.15)
+			)
+			(justify bottom)
+		)
+	)
+	(gr_text "github.com/gcormier/serialsentinel\nv1"
 		(at 49.778402 66.496847 0)
 		(layer "F.SilkS")
@@
 	)
 	(gr_text "Serial Sentinel"
-		(at 49.778402 64.478217 0)
+		(at 49.777853 62.441931 0)
 		(layer "F.SilkS")
 		(effects
@@
 		)
 	)
+	(gr_text "JLCJLCJLCJLC"
+		(at 49.895825 79.252922 0)
+		(layer "F.SilkS")
+		(effects
+			(font
+				(size 1 1)
+				(thickness 0.15)
+			)
+			(justify bottom)
+		)
+	)
 	(gr_text "GPIO6"
 		(at 90.265 82.23 0)
@@
 	)
 	(segment
-		(start 65.725 79.35)
-		(end 63.785931 79.35)
+		(start 64.908074 63.5)
+		(end 65.525 63.5)
 		(width 0.2)
 		(layer "F.Cu")
@@
 	)
 	(segment
-		(start 49.11 82.2)
-		(end 47.8 82.2)
+		(start 65.725 79.35)
+		(end 63.785931 79.35)
 		(width 0.2)
 		(layer "F.Cu")
@@
 	)
 	(segment
-		(start 63.672836 63.5)
-		(end 63.612523 63.439687)
+		(start 49.11 82.2)
+		(end 47.8 82.2)
 		(width 0.2)
 		(layer "F.Cu")
@@
 	)
 	(segment
-		(start 65.525 63.5)
-		(end 63.672836 63.5)
-		(width 0.2)
-		(layer "F.Cu")
-		(net 1)
-	)
-	(segment
 		(start 67.8 85.176554)
 		(end 68.257883 85.634437)
@@
 	)
 	(segment
+		(start 63.92137 62.513296)
+		(end 64.908074 63.5)
+		(width 0.2)
+		(layer "F.Cu")
+		(net 1)
+	)
+	(segment
 		(start 56 93)
 		(end 56 91.224737)
@@
 	)
 	(via
-		(at 63.612523 63.439687)
+		(at 63.92137 62.513296)
 		(size 0.8)
 		(drill 0.4)
@@
 	)
 	(segment
-		(start 66.376799 60.03928)
-		(end 66.376799 60.748201)
+		(start 68 61)
+		(end 67.748201 60.748201)
 		(width 0.2)
 		(layer "F.Cu")
@@
 		(net 52)
 	)
+	(segment
+		(start 67.748201 60.748201)
+		(end 66.376799 60.748201)
+		(width 0.2)
+		(layer "F.Cu")
+		(net 52)
+	)
 	(via
-		(at 66.376799 60.03928)
+		(at 68 61)
 		(size 0.8)
 		(drill 0.4)
@@
 	)
 	(segment
+		(start 66.376799 62.623201)
+		(end 68 61)
+		(width 0.2)
+		(layer "B.Cu")
+		(net 52)
+	)
+	(segment
 		(start 66.376799 70.032312)
-		(end 66.376799 60.03928)
+		(end 66.376799 62.623201)
 		(width 0.2)
 		(layer "B.Cu")
@@
 			(thermal_gap 0.508)
 			(thermal_bridge_width 0.508)
+			(smoothing fillet)
+			(radius 0.25)
 		)
 		(polygon
 			(pts
-				(xy 23.37187 58.643188) (xy 96.49687 58.643188) (xy 96.49687 114.768188) (xy 88.74687 114.768188)
+				(xy 24.37187 59.643188) (xy 95.49687 59.643188) (xy 95.49687 113.768188) (xy 88.74687 113.768188)
 				(xy 88.74687 121.918188) (xy 68.24687 121.918188) (xy 68.24687 116.643188) (xy 64.74687 116.643188)
-				(xy 64.74687 116.179484) (xy 56.62187 116.179484) (xy 56.62187 114.768188) (xy 38.37187 114.768188)
-				(xy 38.37187 123.018188) (xy 23.37187 123.018188)
+				(xy 64.74687 116.179484) (xy 57.62187 116.179484) (xy 57.62187 113.768188) (xy 37.37187 113.768188)
+				(xy 37.37187 122.018188) (xy 24.37187 122.018188)
 			)
 		)

Commit message: tweaks
Parts:
- added D5: NCD0805R1, LED_SMD:LED_0805_2012Metric, F.Cu at (48.6, 62.0)
- added D6: NCD0805R1, LED_SMD:LED_0805_2012Metric, F.Cu at (56.4, 62.0)
- added D7: NCD0805R1, LED_SMD:LED_0805_2012Metric, F.Cu at (40.6, 62.0)
- added R10: 1k, Resistor_SMD:R_0402_1005Metric, F.Cu at (59.4, 62.0)
- added R14: 1k, Resistor_SMD:R_0402_1005Metric, F.Cu at (43.6, 62.0)
- added R9: 1k, Resistor_SMD:R_0402_1005Metric, F.Cu at (51.6, 62.0)
Connections:
- U3 pad 10: unconnected-(U3-IO10-Pad10) -> LED3
- U3 pad 18: unconnected-(U3-IO0-Pad18) -> LED1
- U3 pad 6: unconnected-(U3-IO7-Pad6) -> LED2
Routing:
- net LED2: track 0.00 -> 38.6 mm, vias 0 -> 2
- net LED1: track 0.00 -> 17.7 mm, vias 0 -> 2
- net LED3: track 0.00 -> 13.7 mm
- net GND: track 96.8 -> 99.7 mm, vias 42 -> 45
- net Net-(D6-K): track 0.00 -> 1.55 mm
- net Net-(D5-K): track 0.00 -> 1.55 mm
- net Net-(D7-K): track 0.00 -> 1.49 mm
Other:
- board text added: "Edge Connector - hard gold + edge bevel Do NOT place mousebites for panel."
- board text added: "LED1"
- board text added: "LED2"
- board text added: "LED3"
- board text removed: "Edge Connector - hard gold + edge bevel"
