File: pcb/serialsentinel.kicad_pcb (KiCad board)
At the start: 4 copper layers, 73.2 x 64.4 mm, 45 parts, among them J2 Bus_PCI_Express_x1, J3 REL1, J4 REL1, J5 REL2, J6 REL2, K2 G6K-2F-Y DC3, K3 G6K-2F-Y DC3, Q2 MMBT3904, Q3 MMBT3904, Q4 MMBT3904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

Commit message: touchup
Routing:
- net U0_DTR: track 42.6 -> 64.3 mm, vias 2 -> 4
- net GND: track 99.7 -> 104.9 mm
- net U0_RTS: track 78.3 -> 80.8 mm
- net U1_TX: track 54.6 -> 56.4 mm
Other:
- board text added: "LED1 GPIO0"
- board text added: "LED2 GPIO7"
- board text added: "LED3 GPIO10"
- board text added: "github.com/gcormier/serialsentinel <<hash>>"
- board text removed: "<<hash>>"
- board text removed: "LED1"
- board text removed: "LED2"
- board text removed: "LED3"
- board text removed: "github.com/gcormier/serialsentinel v1"

Commit message: final tweaks
Parts:
- removed D6: NCD0805R1, LED_SMD:LED_0805_2012Metric
- removed R10: 1k, Resistor_SMD:R_0402_1005Metric
- added C4: 100n, Capacitor_SMD:C_0402_1005Metric, F.Cu at (80.7, 107.2)
- added C5: 100n, Capacitor_SMD:C_0402_1005Metric, F.Cu at (78.4, 95.0)
- added C6: 100n, Capacitor_SMD:C_0402_1005Metric, F.Cu at (89.2, 106.4)
- added C7: 100n, Capacitor_SMD:C_0402_1005Metric, F.Cu at (89.8, 102.6)
- added C8: 100n, Capacitor_SMD:C_0402_1005Metric, F.Cu at (89.8, 96.3)
- added J1: PCIexpress_bracket, PCIexpress:PCIexpress_bracket_low, F.Cu at (68.5, 127.5)
- added JP1: WAKE, Jumper:SolderJumper-2_P1.3mm_Bridged_RoundedPad1.0x1.5mm, B.Cu at (51.5, 112.0)
- moved JP2 2.00 mm to (72.5, 112.0)
Connections:
- J2 pad B11: unconnected-(J2-~{WAKE}-PadB11) -> WAKE
- J2 pad B5: I2C_SCL -> I2C_CLK
- J2 pad B6: I2C_SDA -> I2C_DAT
- U3 pad 10: LED3 -> I2C_CLK
- U3 pad 13: unconnected-(U3-IO18-Pad13) -> I2C_DAT
- U3 pad 14: unconnected-(U3-IO19-Pad14) -> Net-(JP1-B)
Routing:
- net I2C_DAT: track 0.00 -> 71.7 mm, vias 0 -> 2
- net I2C_CLK: track 0.00 -> 64.2 mm, vias 0 -> 2
- net Net-(JP1-B): track 0.00 -> 53.9 mm, vias 0 -> 3
- net +1V8: track 54.9 -> 92.5 mm, vias 3 -> 9
- net WAKE: track 0.00 -> 37.2 mm, vias 0 -> 3
- net +3V3: track 99.9 -> 114.7 mm, vias 8 -> 9
- net LED3: track 13.7 -> 0.00 mm
- net +3V3AUX: track 107.9 -> 112.2 mm, vias 4 -> 6
- net U0_RTS: track 80.8 -> 78.4 mm
- net U0_RX: track 61.5 -> 63.4 mm
- net Net-(D6-K): track 1.55 -> 0.00 mm
- net LED2: track 38.6 -> 40.1 mm, vias 2 -> 4
- net Net-(J2-~{PRSNT1}): track 11.9 -> 13.2 mm
- net GND: track 104.9 -> 104.1 mm, vias 45 -> 52
- net U0_DTR: track 64.3 -> 63.7 mm
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Other:
- board text added: "Dielectric Constant 4.4 Eff = 3.33"
- board text added: "GPIO10 I2C_CLK GPIO18 I2C_DAT GPIO19 WAKE"
- board text added: "Stackup JLC04161H-7628 Material FR4 TG155"
- board text removed: "LED3 GPIO10"

Commit message: fix footprint
Parts:
- R12, R2, R206, R4, R5, R6: value 10k -> 12K
Changed lines of the file:
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@@
 			)
 		)
-		(property "Value" "10k"
+		(property "Value" "12K"
 			(at 0 1.17 90)
 			(layer "F.Fab")
@@
 			)
 		)
-		(property "Description" ""
+		(property "Description" "Resistor, small symbol"
 			(at 0 0 90)
 			(layer "F.Fab")
@@
 			)
 		)
-		(property "LCSC" "C25744"
+		(property "LCSC" "C25752"
 			(at 0 0 90)
 			(unlocked yes)
@@
 			)
 		)
-		(property "Description" ""
+		(property "Description" "Light emitting diode, small symbol"
 			(at 0 0 0)
 			(layer "F.Fab")
@@
 			)
 		)
+		(property "Sim.Pin" "1=K 2=A"
+			(at 0 0 180)
+			(unlocked yes)
+			(layer "F.Fab")
+			(hide yes)
+			(effects
+				(font
+					(size 1 1)
+					(thickness 0.15)
+				)
+			)
+		)
 		(property ki_fp_filters "LED* LED_SMD:* LED_THT:*")
 		(sheetname "/")
@@
 			)
 		)
-		(property "Value" "10k"
+		(property "Value" "12K"
 			(at 0 1.17 0)
 			(layer "F.Fab")
@@
 			)
 		)
-		(property "Description" ""
+		(property "Description" "Resistor, small symbol"
 			(at 0 0 0)
 			(layer "F.Fab")
@@
 			)
 		)
-		(property "LCSC" "C25744"
+		(property "LCSC" "C25752"
 			(at 0 0 180)
 			(unlocked yes)
@@
 			)
 		)
-		(property "Description" ""
+		(property "Description" "Light emitting diode, small symbol"
 			(at 0 0 0)
 			(layer "F.Fab")
@@
 			)
 		)
+		(property "Sim.Pin" "1=K 2=A"
+			(at 0 0 180)
+			(unlocked yes)
+			(layer "F.Fab")
+			(hide yes)
+			(effects
+				(font
+					(size 1 1)
+					(thickness 0.15)
+				)
+			)
+		)
 		(property ki_fp_filters "LED* LED_SMD:* LED_THT:*")
 		(sheetname "/")
@@
 			)
 		)
-		(property "Description" ""
+		(property "Description" "Resistor, small symbol"
 			(at 0 0 0)
 			(layer "F.Fab")
@@
 			)
 		)
-		(property "LCSC" "C21190"
+		(property "LCSC" "C11702"
 			(at 0 0 0)
 			(unlocked yes)
@@
 			)
 		)
-		(property "Description" ""
+		(property "Description" "Resistor, small symbol"
 			(at 0 0 90)
 			(layer "F.Fab")
@@
 			)
 		)
-		(property "LCSC" "C21190"
+		(property "LCSC" "C11702"
 			(at 0 0 270)
 			(unlocked yes)
@@
 			)
 		)
-		(property "Description" ""
+		(property "Description" "Resistor, small symbol"
 			(at 0 0 90)
 			(layer "F.Fab")
@@
 			)
 		)
-		(property "LCSC" "C21190"
+		(property "LCSC" "C11702"
 			(at 0 0 270)
 			(unlocked yes)
@@
 			)
 		)
-		(property "Description" ""
+		(property "Description" "Resistor, small symbol"
 			(at 0 0 0)
 			(layer "F.Fab")
@@
 			)
 		)
-		(property "LCSC" "C21190"
+		(property "LCSC" "C11702"
 			(at 0 0 0)
 			(unlocked yes)
@@
 			)
 		)
-		(property "Description" ""
+		(property "Description" "Light emitting diode, small symbol"
 			(at 0 0 0)
 			(layer "F.Fab")
@@
 			)
 		)
+		(property "Sim.Pin" "1=K 2=A"
+			(at 0 0 180)
+			(unlocked yes)
+			(layer "F.Fab")
+			(hide yes)
+			(effects
+				(font
+					(size 1 1)
+					(thickness 0.15)
+				)
+			)
+		)
 		(property ki_fp_filters "LED* LED_SMD:* LED_THT:*")
 		(sheetname "/")
@@
 			)
 		)
-		(property "Description" ""
+		(property "Description" "Light emitting diode, small symbol"
 			(at 0 0 0)
 			(layer "F.Fab")
@@
 			)
 		)
+		(property "Sim.Pin" "1=K 2=A"
+			(at 0 0 180)
+			(unlocked yes)
+			(layer "F.Fab")
+			(hide yes)
+			(effects
+				(font
+					(size 1 1)
+					(thickness 0.15)
+				)
+			)
+		)
 		(property ki_fp_filters "LED* LED_SMD:* LED_THT:*")
 		(sheetname "/")
@@
 			)
 		)
-		(property "Description" ""
+		(property "Description" "Resistor, small symbol"
 			(at 0 0 0)
 			(layer "F.Fab")
@@
 			)
 		)
-		(property "LCSC" "C21190"
+		(property "LCSC" "C11702"
 			(at 0 0 180)
 			(unlocked yes)
@@
 			)
 		)
-		(property "Value" "10k"
+		(property "Value" "12K"
 			(at 0 1.17 90)
 			(layer "F.Fab")
@@
 			)
 		)
-		(property "Description" ""
+		(property "Description" "Resistor, small symbol"
 			(at 0 0 90)
 			(layer "F.Fab")
@@
 			)
 		)
-		(property "LCSC" "C25744"
+		(property "LCSC" "C25752"
 			(at 0 0 270)
 			(unlocked yes)
@@
 			)
 		)
-		(property "Value" "10k"
+		(property "Value" "12K"
 			(at 0 1.17 0)
 			(layer "F.Fab")
@@
 			)
 		)
-		(property "Description" ""
+		(property "Description" "Resistor, small symbol"
 			(at 0 0 0)
 			(layer "F.Fab")
@@
 			)
 		)
-		(property "LCSC" "C25744"
+		(property "LCSC" "C25752"
 			(at 0 0 180)
 			(unlocked yes)
@@
 			)
 		)
-		(property "Description" ""
+		(property "Description" "Resistor, small symbol"
 			(at 0 0 90)
 			(layer "F.Fab")
@@
 			)
 		)
-		(property "LCSC" "C21190"
+		(property "LCSC" "C11702"
 			(at 0 0 270)
 			(unlocked yes)
@@
 			)
 		)
-		(property "Description" ""
+		(property "Description" "Resistor, small symbol"
 			(at 0 0 90)
 			(layer "F.Fab")
@@
 			)
 		)
-		(property "LCSC" "C21190"
+		(property "LCSC" "C11702"
 			(at 0 0 270)
 			(unlocked yes)
@@
 			)
 		)
-		(property "Value" "10k"
+		(property "Value" "12K"
 			(at 0 1.17 90)
 			(layer "F.Fab")
@@
 			)
 		)
-		(property "Description" ""
+		(property "Description" "Resistor, small symbol"
 			(at 0 0 90)
 			(layer "F.Fab")
@@
 			)
 		)
-		(property "LCSC" "C25744"
+		(property "LCSC" "C25752"
 			(at 0 0 90)
 			(unlocked yes)
@@
 			)
 		)
-		(property "Value" "10k"
+		(property "Value" "12K"
 			(at 0 1.17 90)
 			(layer "F.Fab")
@@
 			)
 		)
-		(property "Description" ""
+		(property "Description" "Resistor, small symbol"
 			(at 0 0 90)
 			(layer "F.Fab")
@@
 			)
 		)
-		(property "LCSC" "C25744"
+		(property "LCSC" "C25752"
 			(at 0 0 270)
 			(unlocked yes)

Commit message: fixes
Parts:
- added J7: eflashy32, Connector_PinHeader_2.54mm:PinHeader_1x06_P2.54mm_Vertical, F.Cu at (49.8, 54.2)
- moved Q3 30.1 mm to (82.4, 52.7)
- moved Q4 30.1 mm to (59.9, 43.7)
- moved C213 30.1 mm to (59.2, 69.3)
- moved C214 30.1 mm to (96.8, 66.8)
- moved C217 30.1 mm to (83.9, 80.3)
- moved C4 30.1 mm to (96.4, 81.5)
- moved D1 30.1 mm to (86.3, 39.8)
- moved D2 30.1 mm to (86.4, 55.6)
- moved D5 30.1 mm to (64.3, 36.3)
- moved D7 30.1 mm to (56.4, 36.3)
- moved J3 30.1 mm to (101.9, 35.0)
- moved J4 30.1 mm to (101.9, 42.1)
- moved J5 30.1 mm to (101.9, 50.8)
- moved J6 30.1 mm to (101.9, 57.9)
- moved JP1 30.1 mm to (67.3, 86.3)
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Connections:
- U1 pad 11: PER+ -> PET+
- U1 pad 12: PER- -> PET-
- U1 pad 14: PET+ -> PER+
- U1 pad 15: PET- -> PER-
Routing:
- net GPIO0: track 27.1 -> 51.5 mm, vias 0 -> 2
- net +3V3: track 114.7 -> 137.6 mm, vias 9 -> 10
- net U0_TX: track 46.6 -> 67.6 mm, vias 2 -> 4
- net U0_RX: track 63.4 -> 83.2 mm, vias 2 -> 4
- net EN: track 34.3 -> 40.8 mm
- net GND: track 104.1 -> 102.7 mm, vias 52 -> 51
- net PER-: track 21.9 -> 20.5 mm
- net PET-: track 21.0 -> 22.4 mm
- net PET+: track 21.0 -> 22.4 mm
- net PER+: track 21.9 -> 20.7 mm
Other:
- outline, holes or cut-outs redrawn

Commit message: towards v3!
Parts:
- added C3: 220n, Capacitor_SMD:C_0402_1005Metric, F.Cu at (101.1, 86.5)
- added C9: 220n, Capacitor_SMD:C_0402_1005Metric, F.Cu at (102.1, 86.5)
- added D6: NCD0805R1, LED_SMD:LED_0805_2012Metric, F.Cu at (71.7, 36.2)
- added J8: BOOTSEL, Connector_PinHeader_2.54mm:PinHeader_1x02_P2.54mm_Vertical, F.Cu at (62.8, 79.1)
- added JP3: CrystalMode, Jumper:SolderJumper-3_P1.3mm_Bridged12_RoundedPad1.0x1.5mm, B.Cu at (93.2, 78.2)
- added R10: 12K, Resistor_SMD:R_0402_1005Metric, F.Cu at (96.3, 90.3)
- added R15: 1k, Resistor_SMD:R_0402_1005Metric, F.Cu at (74.8, 36.2)
- J1: value PCIexpress_bracket -> BRIDGE3V; footprint PCIexpress:PCIexpress_bracket_low -> Connector_PinHeader_2.54mm:PinHeader_1x02_P2.54mm_Vertical
- moved J1 39.4 mm to (52.5, 78.5), turned to 90 degrees
Connections:
- J2 pad B12: unconnected-(J2-RSVD-PadB12) -> /CLKREQ
- J7 pad 4: +3V3 -> +3V3AUX
- U1 pad 14: PER+ -> /PRC+
- U1 pad 15: PER- -> /PRC-
- U1 pad 64: unconnected-(U1-CKSEL-Pad64) -> CKSEL
Routing:
- net +3V3AUX: track 112.2 -> 138.4 mm, vias 6 -> 7
- net +3V3: track 137.6 -> 123.3 mm
- net PER+: track 20.7 -> 12.1 mm
- net PER-: track 20.5 -> 12.0 mm
- net /CLKREQ: track 0.00 -> 8.18 mm
- net /PRC+: track 0.00 -> 7.85 mm
- net /PRC-: track 0.00 -> 7.85 mm
- net GND: track 102.7 -> 105.9 mm, vias 51 -> 52
- net CKSEL: track 0.00 -> 2.89 mm, vias 0 -> 1
- net Net-(J2-~{PRSNT2}): track 26.0 -> 28.2 mm
- net GPIO0: track 51.5 -> 53.4 mm
- net PERST: track 21.4 -> 23.0 mm
- net PET+: track 22.4 -> 23.0 mm
- net PET-: track 22.4 -> 23.0 mm
Other:
- board text added: "AUX PWR"
- board text added: "GND RX TX 3VAUX EN GPIO9"

Commit message: ayo
Parts:
- added BZ1: Buzzer, Buzzer_Beeper:MagneticBuzzer_PUI_AT-0927-TT-6-R, B.Cu at (68.3, 41.7)
- added C10: 22u, Capacitor_SMD:C_0603_1608Metric, F.Cu at (113.9, 78.0)
- added D10: Green, LED_SMD:LED_0805_2012Metric, F.Cu at (76.9, 36.2)
- added D8: SS54, Diode_SMD:D_SMA, F.Cu at (94.4, 87.7)
- added D9: SS54, Diode_SMD:D_SMA, F.Cu at (90.9, 87.7)
- added J9: EXTPWR, Connector_TE-Connectivity:TE_2834006-2_1x02_P4.0mm_Horizontal, F.Cu at (113.7, 70.0)
- added JP4: RP3VAUX, Jumper:SolderJumper-2_P1.3mm_Open_RoundedPad1.0x1.5mm, B.Cu at (94.4, 87.7)
- added JP5: RP3V, Jumper:SolderJumper-2_P1.3mm_Open_RoundedPad1.0x1.5mm, B.Cu at (91.4, 87.7)
- added JP6: ESP32PWR, Jumper:SolderJumper-3_P1.3mm_Bridged12_RoundedPad1.0x1.5mm, B.Cu at (55.8, 74.0)
- added R16: 1k, Resistor_SMD:R_0402_1005Metric, F.Cu at (74.1, 39.6)
- added U4: AMS1117-3.3, Package_TO_SOT_SMD:SOT-223-3_TabPin2, F.Cu at (113.1, 84.0)
- D3, D4, D5, D6, D7: value NCD0805R1 -> Red
- moved C217 13.1 mm to (90.4, 91.7), turned to 0 degrees
- moved J3 8.26 mm to (110.1, 35.0)
- moved J4 8.26 mm to (110.1, 42.1)
- moved J5 8.26 mm to (110.1, 50.8)
- moved J6 8.26 mm to (110.1, 57.9)
- moved R15 5.84 mm to (79.6, 39.5), turned to -90 degrees
- moved R10 1.76 mm to (97.4, 91.7)
- moved JP2 0.63 mm to (87.6, 86.3)
- moved C8 0.44 mm to (105.1, 70.5)
- moved D6 0.31 mm to (71.4, 36.2)
Connections:
- C213 pad 2: +3V3AUX -> Net-(JP6-C)
- C216 pad 2: +3V3AUX -> +3V3AUX_UNPROT
- C217 pad 2: +3V3 -> +3V3_UNPROT
- D6 pad 2: +3V3AUX -> +3V3_UNPROT
- J2 pad A10: +3V3 -> +3V3_UNPROT
- J2 pad A9: +3V3 -> +3V3_UNPROT
- J2 pad B10: +3V3AUX -> +3V3AUX_UNPROT
- J2 pad B8: +3V3 -> +3V3_UNPROT
- R15 pad 1: Net-(D6-K) -> Net-(D10-K)
- U3 pad 1: +3V3AUX -> Net-(JP6-C)
Routing:
- net +3V3_UNPROT: track 0.00 -> 87.5 mm, vias 0 -> 4
- net +3V3AUX_UNPROT: track 0.00 -> 80.1 mm, vias 0 -> 7
- net +3V3AUX: track 138.4 -> 191.8 mm, vias 7 -> 9
- net /5V_EXT: track 0.00 -> 20.7 mm, vias 0 -> 2
- net Net-(J5-Pin_2): track 17.0 -> 33.5 mm
- net Net-(J3-Pin_2): track 17.1 -> 33.5 mm
- net Net-(J5-Pin_1): track 12.8 -> 28.4 mm
- net +3V3: track 123.3 -> 107.6 mm
- net Net-(J3-Pin_1): track 13.4 -> 28.9 mm
- net LED1: track 17.7 -> 29.0 mm
- net Net-(JP6-C): track 0.00 -> 8.96 mm, vias 0 -> 1
- net GND: track 105.9 -> 111.2 mm, vias 52 -> 56
- net Net-(D6-K): track 0.00 -> 4.20 mm
- net Net-(D10-K): track 0.00 -> 3.47 mm
- net /CLKREQ: track 8.18 -> 6.32 mm
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Other:
- board size 73.2 x 64.4 mm -> 82 x 64.4 mm
- board text added: "- Always turn off main power source when working with this board - Check for AUX PWR LED when PC is off - If required, supply either 5V_EXT or 3V3_EXT - Do NOT supply both"
- board text added: "3V PWR"
- board text added: "3V3 EXT"
- board text added: "4mm pin spacing"
- board text added: "5V EXT"
- board text added: "DO NOT > USE BOTH >"

Commit message: fix diode val
Parts:
- D1, D2: value M7 -> SS54
Changed lines of the file:
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@@
 			)
 		)
+		(property "LCSC" "C6186"
+			(at 0 0 270)
+			(unlocked yes)
+			(layer "F.Fab")
+			(hide yes)
+			(effects
+				(font
+					(size 1 1)
+					(thickness 0.15)
+				)
+			)
+		)
+		(property "Notes" ""
+			(at 0 0 270)
+			(unlocked yes)
+			(layer "F.Fab")
+			(hide yes)
+			(effects
+				(font
+					(size 1 1)
+					(thickness 0.15)
+				)
+			)
+		)
 		(property ki_fp_filters "SOT?223*TabPin2*")
 		(sheetname "/")
@@
 			)
 		)
-		(property "Value" "M7"
+		(property "Value" "SS54"
 			(at 0 2.6 90)
 			(layer "F.Fab")
@@
 			)
 		)
-		(property "Value" "M7"
+		(property "Value" "SS54"
 			(at 0 2.6 90)
 			(layer "F.Fab")

Commit message: fix things
Parts:
- removed JP2: PRSNT, Jumper:SolderJumper-2_P1.3mm_Bridged_RoundedPad1.0x1.5mm
- added C11: 10u, Capacitor_SMD:C_0402_1005Metric, F.Cu at (93.1, 69.3)
- added C12: 10u, Capacitor_SMD:C_0402_1005Metric, F.Cu at (88.9, 78.7)
- added C13: 100n, Capacitor_SMD:C_0402_1005Metric, F.Cu at (92.7, 74.4)
- added C14: 10u, Capacitor_SMD:C_0402_1005Metric, F.Cu at (96.4, 81.4)
- added R17: 1k, Resistor_SMD:R_0402_1005Metric, F.Cu at (76.6, 56.5)
- added R18: 1k, Resistor_SMD:R_0402_1005Metric, F.Cu at (94.8, 62.5)
- added R19: 1k, Resistor_SMD:R_0402_1005Metric, F.Cu at (76.6, 61.0)
- added R20: 1k, Resistor_SMD:R_0402_1005Metric, F.Cu at (92.6, 62.5)
- C3, C9: value 220n -> 100n
- J3: value REL1 -> DTR; footprint Connector_PinHeader_2.54mm:PinHeader_1x02_P2.54mm_Horizontal -> Connector_PinHeader_2.54mm:PinHeader_1x02_P2.54mm_Vertical
- J4: value REL1 -> RTS; footprint Connector_PinHeader_2.54mm:PinHeader_1x02_P2.54mm_Horizontal -> Connector_PinHeader_2.54mm:PinHeader_1x02_P2.54mm_Vertical
- J5: value REL2 -> RELAY1; footprint Connector_PinHeader_2.54mm:PinHeader_1x02_P2.54mm_Horizontal -> Connector_PinHeader_2.54mm:PinHeader_1x05_P2.54mm_Horizontal
- J6: value REL2 -> RELAY2; footprint Connector_PinHeader_2.54mm:PinHeader_1x02_P2.54mm_Horizontal -> Connector_PinHeader_2.54mm:PinHeader_1x05_P2.54mm_Horizontal
- moved J3 58.2 mm to (52.9, 45.5)
- moved J4 57.0 mm to (70.4, 83.0), turned to 180 degrees
- moved J5 15.6 mm to (110.0, 35.2)
- moved R8 14.2 mm to (100.7, 67.7), turned to 0 degrees
- moved J6 7.46 mm to (110.0, 50.5)
- moved C4 1.15 mm to (96.4, 80.4)
- moved C6 0.54 mm to (105.1, 80.2)
Connections:
- J2 pad B17: Net-(J2-~{PRSNT2}) -> Net-(J2-~{PRSNT1})
- J3 pad 2: Net-(J3-Pin_2) -> EN
- J4 pad 1: Net-(J3-Pin_1) -> GPIO0
- J4 pad 2: Net-(J3-Pin_2) -> Net-(J4-Pin_2)
- J6 pad 1: Net-(J5-Pin_1) -> Net-(J6-Pin_1)
- J6 pad 2: Net-(J5-Pin_2) -> Net-(J6-Pin_2)
- K2 pad 5: Net-(J3-Pin_1) -> Net-(J5-Pin_1)
- K2 pad 6: Net-(J3-Pin_2) -> Net-(J5-Pin_2)
- K3 pad 5: Net-(J5-Pin_1) -> Net-(J6-Pin_1)
- K3 pad 6: Net-(J5-Pin_2) -> Net-(J6-Pin_2)
- Q4 pad 3: EN -> Net-(J3-Pin_1)
- Q5 pad 3: GPIO0 -> Net-(J4-Pin_2)
- R206 pad 1: +3V3 -> Net-(JP6-C)
- U1 pad 27: U0_RX -> Net-(U1-RXD0)
- U1 pad 34: U1_RX -> Net-(U1-RXD1)
- U1 pad 50: U0_TX -> Net-(U1-TXD0)
- U1 pad 53: U1_TX -> Net-(U1-TXD1)
Routing:
- net Net-(U1-RXD0): track 0.00 -> 50.2 mm, vias 0 -> 4
- net U0_RX: track 81.4 -> 33.9 mm, vias 4 -> 3
- net Net-(J6-Pin_2): track 0.00 -> 33.8 mm, vias 0 -> 1
- net Net-(J3-Pin_2): track 33.5 -> 0.00 mm, vias 1 -> 0
- net Net-(J2-~{PRSNT1}): track 13.0 -> 43.7 mm, vias 0 -> 1
- net U0_TX: track 67.6 -> 38.6 mm, vias 4 -> 3
- net Net-(J2-~{PRSNT2}): track 28.9 -> 0.00 mm, vias 1 -> 0
- net Net-(J6-Pin_1): track 0.00 -> 28.4 mm
- net Net-(U1-TXD0): track 0.00 -> 27.6 mm, vias 0 -> 2
- net Net-(J3-Pin_1): track 28.9 -> 7.37 mm, vias 0 -> 1
- net U1_TX: track 56.5 -> 43.6 mm
- net Net-(U1-RXD1): track 0.00 -> 12.9 mm
- net Net-(U1-TXD1): track 0.00 -> 12.8 mm, vias 0 -> 2
- net +1V8: track 91.1 -> 100.9 mm, vias 9 -> 13
- net Net-(J4-Pin_2): track 0.00 -> 8.33 mm
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