File: pcb/serialsentinel.kicad_pcb (KiCad board)
At the start: 4 copper layers, 82 x 64.4 mm, 76 parts, among them J1 BRIDGE3V, J2 Bus_PCI_Express_x1, J3 DTR, J4 RTS, J5 RELAY1, J6 RELAY2, J7 eflashy32, J8 BOOTSEL, J9 EXTPWR, K2 G6K-2F-Y DC3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

Commit message: changes based on review pt 1
Parts:
- removed D5: Red, LED_SMD:LED_0805_2012Metric
- removed J1: BRIDGE3V, Connector_PinHeader_2.54mm:PinHeader_1x02_P2.54mm_Vertical
- removed JP3: CrystalMode, Jumper:SolderJumper-3_P1.3mm_Bridged12_RoundedPad1.0x1.5mm
- removed JP6: ESP32PWR, Jumper:SolderJumper-3_P1.3mm_Bridged12_RoundedPad1.0x1.5mm
- removed R9: 1k, Resistor_SMD:R_0402_1005Metric
- added C15: 1u, Capacitor_SMD:C_0402_1005Metric, F.Cu at (62.3, 70.8)
- J9: value EXTPWR -> 5VEXT; footprint Connector_TE-Connectivity:TE_2834006-2_1x02_P4.0mm_Horizontal -> Connector_PinHeader_2.54mm:PinHeader_1x02_P2.54mm_Vertical
- moved R15 44.0 mm to (107.3, 73.7), turned to 180 degrees
- moved D10 43.7 mm to (107.1, 67.9)
- moved C2 21.8 mm to (95.3, 70.1), turned to -90 degrees
- moved C214 21.8 mm to (96.6, 88.7)
- moved C12 18.0 mm to (106.8, 79.7), turned to -90 degrees
- moved C1 17.3 mm to (94.4, 73.1), turned to 0 degrees
- moved U2 16.4 mm to (92.5, 70.6), turned to 180 degrees
- moved C8 16.3 mm to (106.2, 86.7), turned to 90 degrees
- moved R8 15.6 mm to (107.1, 81.9)
- moved C14 12.0 mm to (107.2, 86.7), turned to -90 degrees
- moved R6 11.5 mm to (89.1, 76.9)
- moved R7 11.5 mm to (89.1, 75.7)
- moved JP4 10.6 mm to (85.5, 81.9)
- moved C215 9.75 mm to (94.5, 87.5), turned to 0 degrees
- moved D8 9.10 mm to (87.3, 82.0)
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Connections:
- BZ1 pad 1: LED1 -> BUZZ1
- C213 pad 2: Net-(JP6-C) -> +3V3AUX
- J2 pad A11: PERST -> CKSEL
- J2 pad B5: I2C_CLK -> unconnected-(J2-SMCLK-PadB5)
- J2 pad B6: I2C_DAT -> unconnected-(J2-SMDAT-PadB6)
- J9 pad 2: +3V3AUX -> /5V_EXT
- R206 pad 1: Net-(JP6-C) -> +3V3AUX
- U1 pad 1: PERST -> CKSEL
- U3 pad 1: Net-(JP6-C) -> +3V3AUX
- U3 pad 10: I2C_CLK -> BUZZ1
- U3 pad 13: I2C_DAT -> unconnected-(U3-IO18-Pad13)
- U3 pad 6: LED2 -> unconnected-(U3-IO7-Pad6)
Routing:
- net +3V3AUX: track 185.5 -> 112.3 mm, vias 9 -> 5
- net I2C_DAT: track 71.7 -> 0.00 mm, vias 2 -> 0
- net +3V3AUX_UNPROT: track 79.4 -> 10.1 mm, vias 7 -> 1
- net I2C_CLK: track 64.2 -> 0.00 mm, vias 2 -> 0
- net Net-(U1-RXD0): track 50.2 -> 0.00 mm, vias 4 -> 0
- net LED2: track 40.4 -> 0.00 mm, vias 4 -> 0
- net +3V3: track 103.1 -> 63.5 mm, vias 8 -> 3
- net unconnected-(U3-IO7-Pad6): track 0.00 -> 38.7 mm, vias 0 -> 3
- net U0_RTS: track 77.7 -> 49.7 mm, vias 3 -> 2
- net Net-(U1-TXD0): track 27.6 -> 0.00 mm, vias 2 -> 0
- net +1V8: track 100.9 -> 74.9 mm, vias 13 -> 8
- net PERST: track 24.3 -> 0.00 mm, vias 3 -> 0
- net U0_DTR: track 63.7 -> 42.0 mm, vias 4 -> 2
- net GND: track 115.6 -> 100.7 mm, vias 59 -> 58
- net /PWR_DET: track 39.2 -> 53.1 mm, vias 2 -> 4
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Other:
- board text added: "2mm max component height"
- board text added: "GPIO19 WAKE"
- board text added: "No components"
- board text removed: "3V3 EXT"
- board text removed: "DO NOT > USE BOTH >"
- board text removed: "GPIO10 I2C_CLK GPIO18 I2C_DAT GPIO19 WAKE"
- board text removed: "LED2 GPIO7"

Commit message: final changes
Parts:
- moved R15 53.6 mm to (68.4, 36.8), turned to -90 degrees
- moved D10 52.7 mm to (64.9, 36.3)
- moved BZ1 4.13 mm to (68.3, 45.8), turned to 90 degrees
- moved R16 2.75 mm to (74.4, 36.8)
- moved R8 1.43 mm to (108.5, 81.9)
- moved R14 1.17 mm to (60.4, 36.8), turned to -90 degrees
- moved D6 0.07 mm to (71.4, 36.3)
Routing:
- net +3V3AUX_UNPROT: track 10.1 -> 88.3 mm, vias 1 -> 5
- net Net-(U1-RXD0): track 0.00 -> 53.2 mm, vias 0 -> 2
- net +3V3AUX: track 112.3 -> 152.6 mm, vias 5 -> 8
- net unconnected-(U3-IO7-Pad6): track 38.7 -> 0.00 mm, vias 3 -> 0
- net Net-(U1-TXD0): track 0.00 -> 38.6 mm, vias 0 -> 2
- net U0_DTR: track 42.0 -> 72.0 mm, vias 2 -> 4
- net U0_RTS: track 49.7 -> 78.3 mm, vias 2 -> 4
- net Net-(U1-TXD1): track 0.00 -> 26.1 mm, vias 0 -> 4
- net Net-(U1-RXD1): track 0.00 -> 22.6 mm, vias 0 -> 2
- net GND: track 100.7 -> 84.1 mm, vias 58 -> 190
- net (no net): track 11.9 -> 0.00 mm, vias 1 -> 0
- net BUZZ1: track 0.00 -> 6.42 mm
- net +1V8: track 74.9 -> 81.1 mm
- net Net-(D10-K): track 0.00 -> 2.55 mm
- net Net-(D6-K): track 4.20 -> 2.05 mm
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- added copper zone on B.Cu, net GND
- added copper zone on F.Cu, net GND
