File: pcb/serialsentinel.kicad_sch (KiCad schematic)
At the start: 39 parts, among them J2 Bus_PCI_Express_x1, J3 REL1, J4 REL1, J5 REL2, J6 REL2, K2 G6K-2F-Y DC3, K3 G6K-2F-Y DC3, Q2 MMBT3904, Q3 MMBT3904, Q4 MMBT3904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

Commit message: tweaks
Parts:
- added D5, D6, D7: NCD0805R1, LED_SMD:LED_0805_2012Metric, symbol Device:LED_Small
- added R10, R14, R9: 1k, Resistor_SMD:R_0402_1005Metric, symbol Device:R_Small
Connections:
- net GND: now also R10.2, R14.2, R9.2
- net LED3: now reaches U3.10 (IO10)
- net LED3: now also D6.2 (A)
- net LED1: now reaches U3.18 (IO0)
- net LED1: now also D7.2 (A)
- net LED2: now reaches U3.6 (IO7)
- net LED2: now also D5.2 (A)
- new net: D6.1 (K), R10.1
- new net: D5.1 (K), R9.1
- new net: D7.1 (K), R14.1
- no-connect marks 57 -> 54
Other:
- note added: "MCU"
- note added: "Status LED"
- moved on the sheet: C1, C2, C213, C214, C215, C216, C217, D1, D2, D3, D4, J2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

Commit message: final tweaks
Parts:
- removed D6: NCD0805R1, LED_SMD:LED_0805_2012Metric, symbol Device:LED_Small
- removed R10: 1k, Resistor_SMD:R_0402_1005Metric, symbol Device:R_Small
- added C4, C5, C6, C7, C8: 100n, Capacitor_SMD:C_0402_1005Metric, symbol Device:C_Small
- added JP1: WAKE, Jumper:SolderJumper-2_P1.3mm_Bridged_RoundedPad1.0x1.5mm, symbol Jumper:SolderJumper_2_Bridged
Connections:
- net I2C_SDA is gone; now on net I2C_DAT: J2.B6 (SMDAT)
- net LED3 is gone; now on net I2C_CLK: U3.10 (IO10)
- net +1V8: now also C4.2, C6.2, C8.2
- net +3V3: now also C5.2, C7.2
- net GND: now also C4.1, C5.1, C6.1, C7.1, C8.1
- net I2C_DAT: now reaches U3.13 (IO18)
- net at U3.14 (IO19): now also JP1.2 (B)
- net WAKE: now reaches J2.B11 (~{WAKE})
- net WAKE: now also JP1.1 (A)
- net I2C_SCL renamed I2C_CLK
- no-connect marks 54 -> 51
Other:
- note added: "PCIe spec says that the motherboard will provide i2c pullups."
- moved on the sheet: C214, C216, C217, J2, JP2, SW1

Commit message: fix footprint
Parts:
- R1, R11, R13, R14, R3, R7, R9: LCSC C21190 -> C11702
- R12, R2, R206, R4, R5, R6: value 10k -> 12K; LCSC C25744 -> C25752

Commit message: fixes
Parts:
- added J7: eflashy32, Connector_PinHeader_2.54mm:PinHeader_1x06_P2.54mm_Vertical, symbol Connector_Generic:Conn_01x06
- SW1: now fitted
Connections:
- net +3V3: now also J7.4 (Pin_4)
- net EN: now also J7.5 (Pin_5)
- net GND: now also J7.1 (Pin_1)
- net GPIO0: now also J7.6 (Pin_6)
- net PER+: now also U1.14 (PET-); no longer U1.11 (PER+)
- net PER-: now also U1.15 (PET+); no longer U1.12 (PER-)
- net PET+: now also U1.11 (PER+); no longer U1.14 (PET-)
- net PET-: now also U1.12 (PER-); no longer U1.15 (PET+)
- net U0_RX: now also J7.2 (Pin_2)
- net U0_TX: now also J7.3 (Pin_3)
Other:
- note added: "As seen from programmer. Swap RX/TX on this schematic."
- note added: "Programming"

Commit message: towards v3!
Parts:
- added C3, C9: 220n, Capacitor_SMD:C_0402_1005Metric, symbol Device:C_Small
- added D6: NCD0805R1, LED_SMD:LED_0805_2012Metric, symbol Device:LED_Small
- added J1: BRIDGE3V, Connector_PinHeader_2.54mm:PinHeader_1x02_P2.54mm_Vertical, symbol Connector:Conn_01x02_Pin
- added J8: BOOTSEL, Connector_PinHeader_2.54mm:PinHeader_1x02_P2.54mm_Vertical, symbol Connector:Conn_01x02_Pin
- added JP3: CrystalMode, Jumper:SolderJumper-3_P1.3mm_Bridged12_RoundedPad1.0x1.5mm, symbol Jumper:SolderJumper_3_Bridged12
- added R10: 12K, Resistor_SMD:R_0402_1005Metric, symbol Device:R_Small
- added R15: 1k, Resistor_SMD:R_0402_1005Metric, symbol Device:R_Small
Connections:
- net +3V3: now also J1.2 (Pin_2); no longer J7.4 (Pin_4)
- net +3V3AUX: now also J7.4 (Pin_4), D6.2 (A), J1.1 (Pin_1)
- net GND: now also J8.2 (Pin_2), JP3.3 (B), R10.2, R15.2
- net GPIO0: now also J8.1 (Pin_1)
- net PER+: now also C3.1; no longer U1.14 (PET-)
- net PER-: now also C9.1; no longer U1.15 (PET+)
- net PERST: now also JP3.1 (A)
- net CKSEL: now reaches U1.64 (CKSEL)
- net CKSEL: now also JP3.2 (C)
- net CLKREQ: now reaches J2.B12 (RSVD)
- net CLKREQ: now also R10.1
- new net: D6.1 (K), R15.1
- new net PRC+: C3.2, U1.14 (PET-)
- new net PRC-: C9.2, U1.15 (PET+)
- no-connect marks 51 -> 49
Other:
- note added: "Jumpers"
- note added: "Per datasheet"
- moved on the sheet: C1, C2, C213, C214, C215, C217, D1, D2, D3, D4, D5, D7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

Commit message: ayo
Parts:
- added BZ1: Buzzer, Buzzer_Beeper:MagneticBuzzer_PUI_AT-0927-TT-6-R, symbol Device:Buzzer
- added C10: 22u, Capacitor_SMD:C_0603_1608Metric, symbol Device:C_Small
- added D10: Green, LED_SMD:LED_0805_2012Metric, symbol Device:LED_Small
- added D8, D9: SS54, Diode_SMD:D_SMA, symbol Diode:US1A
- added J9: EXTPWR, Connector_TE-Connectivity:TE_2834006-2_1x02_P4.0mm_Horizontal, symbol Connector:Screw_Terminal_01x02
- added JP4: RP3VAUX, Jumper:SolderJumper-2_P1.3mm_Open_RoundedPad1.0x1.5mm, symbol Jumper:Jumper_2_Open
- added JP5: RP3V, Jumper:SolderJumper-2_P1.3mm_Open_RoundedPad1.0x1.5mm, symbol Jumper:Jumper_2_Open
- added JP6: ESP32PWR, Jumper:SolderJumper-3_P1.3mm_Bridged12_RoundedPad1.0x1.5mm, symbol Jumper:SolderJumper_3_Bridged12
- added R16: 1k, Resistor_SMD:R_0402_1005Metric, symbol Device:R_Small
- added U4: AMS1117-3.3, Package_TO_SOT_SMD:SOT-223-3_TabPin2, symbol Regulator_Linear:AMS1117-3.3
- D1, D2: LCSC C95872 -> C22452
- D3, D4, D5, D6, D7: value NCD0805R1 -> Red
- SW1: now not fitted; now left out of the parts list
Connections:
- net +3V3: now also D9.1 (K), JP5.2 (B), JP6.3 (B); no longer C217.2, J2.A10 (+3.3V), J2.A9 (+3.3V), J2.B8 (+3.3V)
- net +3V3AUX: now also C10.1, D8.1 (K), J9.2 (Pin_2), JP4.2 (B), JP6.1 (A), U4.2 (VO); no longer C213.2, C216.2, D6.2 (A), J2.B10 (3.3Vaux), U3.1 (3V3)
- net GND: now also BZ1.2 (-), C10.2, R16.2, U4.1 (GND)
- net LED1: now also BZ1.1 (+)
- net at D6.1 (K): now also R16.1; no longer R15.1
- new net: C213.2, JP6.2 (C), U3.1 (3V3)
- new net: D10.1 (K), R15.1
- new net +3V3AUX_UNPROT: C216.2, D10.2 (A), D8.2 (A), J2.B10 (3.3Vaux), JP4.1 (A)
- new net +3V3_UNPROT: C217.2, D6.2 (A), D9.2 (A), J2.A10 (+3.3V), J2.A9 (+3.3V), J2.B8 (+3.3V), JP5.1 (A)
- new net 5V_EXT: J9.1 (Pin_1), U4.3 (VI)
Other:
- note added: "Power"
- moved on the sheet: D6, J1, JP3, R14, R15, R9

Commit message: add PN for ams
Parts:
- U4: LCSC (none) -> C6186
Changed lines of the file:
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@@
+			)
+		)
+		(property "LCSC" "C6186"
+			(at 130.81 186.69 0)
+			(effects
+				(font
+					(size 1.27 1.27)
+				)
+				(hide yes)
+			)
+		)
+		(property "Notes" ""
+			(at 130.81 186.69 0)
+			(effects
+				(font
+					(size 1.27 1.27)
+				)
+				(hide yes)
 			)
 		)

Commit message: fix diode val
Parts:
- D1, D2: value M7 -> SS54
Changed lines of the file:
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@@
 			)
 		)
-		(property "Value" "M7"
+		(property "Value" "SS54"
 			(at 203.2 140.9699 90)
 			(effects
@@
 			)
 		)
-		(property "Value" "M7"
+		(property "Value" "SS54"
 			(at 179.07 111.7599 90)
 			(effects
