File: pcb/serialsentinel.kicad_sch (KiCad schematic)
At the start: 69 parts, among them J1 BRIDGE3V, J2 Bus_PCI_Express_x1, J3 REL1, J4 REL1, J5 REL2, J6 REL2, J7 eflashy32, J8 BOOTSEL, J9 EXTPWR, K2 G6K-2F-Y DC3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

Commit message: fix things
Parts:
- removed J5, J6: REL2, Connector_PinHeader_2.54mm:PinHeader_1x02_P2.54mm_Horizontal, symbol Connector:Conn_01x02_Pin
- removed JP2: PRSNT, Jumper:SolderJumper-2_P1.3mm_Bridged_RoundedPad1.0x1.5mm, symbol Jumper:SolderJumper_2_Bridged
- added C11, C12, C14: 10u, Capacitor_SMD:C_0402_1005Metric, symbol Device:C_Small
- added C13: 100n, Capacitor_SMD:C_0402_1005Metric, symbol Device:C_Small
- added J5: RELAY1, Connector_PinHeader_2.54mm:PinHeader_1x05_P2.54mm_Horizontal, symbol Connector:Conn_01x05_Pin
- added J6: RELAY2, Connector_PinHeader_2.54mm:PinHeader_1x05_P2.54mm_Horizontal, symbol Connector:Conn_01x05_Pin
- added R17, R18, R19, R20: 1k, Resistor_SMD:R_0402_1005Metric, symbol Device:R_Small
- C3, C9: value 220n -> 100n; LCSC C16772 -> C307331
- J3: value REL1 -> DTR; footprint Connector_PinHeader_2.54mm:PinHeader_1x02_P2.54mm_Horizontal -> Connector_PinHeader_2.54mm:PinHeader_1x02_P2.54mm_Vertical; LCSC C492410 -> C27985187; now fitted
- J4: value REL1 -> RTS; footprint Connector_PinHeader_2.54mm:PinHeader_1x02_P2.54mm_Horizontal -> Connector_PinHeader_2.54mm:PinHeader_1x02_P2.54mm_Vertical; LCSC C492410 -> C27985187; now fitted
Connections:
- net +1V8: now also C12.1, C13.2, C14.1
- net +3V3: now also C11.1; no longer R206.1
- net EN: now also J3.2 (Pin_2); no longer Q4.3 (C)
- net GND: now also C11.2, C12.2, C13.1, C14.2
- net GPIO0: now also J4.1 (Pin_1); no longer Q5.3 (C)
- net U0_RX: now also R17.2; no longer U1.27 (RXD0)
- net U0_TX: now also R19.2; no longer U1.50 (TXD0)
- net U1_RX: now also R18.2; no longer U1.34 (RXD1)
- net U1_TX: now also R20.2; no longer U1.53 (TXD1)
- net at K3.5: now also J6.1 (Pin_1), J6.4 (Pin_4)
- net at K3.6: now also J6.2 (Pin_2), J6.5 (Pin_5)
- net at C213.2, JP6.2 (C), U3.1 (3V3): now also R206.1
- net at J2.A1 (~{PRSNT1}): now also J2.B17 (~{PRSNT2})
- new net: R17.1, U1.27 (RXD0)
- new net: R18.1, U1.34 (RXD1)
- new net: R19.1, U1.50 (TXD0)
- new net: R20.1, U1.53 (TXD1)
- new net: J5.1 (Pin_1), J5.4 (Pin_4), K2.5
- new net: J5.2 (Pin_2), J5.5 (Pin_5), K2.6
- new net: J3.1 (Pin_1), Q4.3 (C)
- new net: J4.2 (Pin_2), Q5.3 (C)
- no-connect marks 49 -> 51
Other:
- moved on the sheet: C217, R206

Commit message: changes based on review pt 1
Parts:
- removed D5: Red, LED_SMD:LED_0805_2012Metric, symbol Device:LED_Small
- removed J1: BRIDGE3V, Connector_PinHeader_2.54mm:PinHeader_1x02_P2.54mm_Vertical, symbol Connector:Conn_01x02_Pin
- removed JP3: CrystalMode, Jumper:SolderJumper-3_P1.3mm_Bridged12_RoundedPad1.0x1.5mm, symbol Jumper:SolderJumper_3_Bridged12
- removed JP6: ESP32PWR, Jumper:SolderJumper-3_P1.3mm_Bridged12_RoundedPad1.0x1.5mm, symbol Jumper:SolderJumper_3_Bridged12
- removed R9: 1k, Resistor_SMD:R_0402_1005Metric, symbol Device:R_Small
- added C15: 1u, Capacitor_SMD:C_0402_1005Metric, symbol Device:C_Small
- J9: value EXTPWR -> 5VEXT; footprint Connector_TE-Connectivity:TE_2834006-2_1x02_P4.0mm_Horizontal -> Connector_PinHeader_2.54mm:PinHeader_1x02_P2.54mm_Vertical; symbol Connector:Screw_Terminal_01x02 -> Connector:Conn_01x02_Pin; LCSC C2765055 -> C27985187
Connections:
- net PERST is gone; now on net CKSEL: J2.A11 (~{PERST}), U1.1 (PERST#)
- net +3V3AUX: now also C213.2, R206.1, U3.1 (3V3); no longer J9.2 (Pin_2)
- net 5V_EXT: now also J9.2 (Pin_2)
- net EN: now also C15.2
- net GND: now also C15.1
- net LED1: no longer BZ1.1 (+)
- net I2C_CLK: no longer names the net of J2.B5 (SMCLK)
- net I2C_CLK: no longer U3.10 (IO10)
- net I2C_DAT: no longer names the net of U3.13 (IO18)
- net I2C_DAT: no longer J2.B6 (SMDAT)
- net LED2: no longer names the net of U3.6 (IO7)
- new net BUZZ1: BZ1.1 (+), U3.10 (IO10)
- no-connect marks 51 -> 55
Other:
- moved on the sheet: BZ1, C213, D10, D6, D7, R14, R15, R16, R206
